File: radio433.kicad_pcb (KiCad board)
At the start: 2 copper layers, 70.5 x 26.8 mm, 31 parts, among them J1 TX, J2 RX, U1 MICRF113YM6-TR, U2 MICRF219AAYQS, Y2 13M52313, Y3 13M56

Commit message: changed shape
Routing:
- net GND: vias 43 -> 40
Other:
- outline, holes or cut-outs redrawn
Changed lines of the file:
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@@
 			(outputformat 1)
 			(mirror no)
-			(drillshape 1)
+			(drillshape 0)
 			(scaleselection 1)
-			(outputdirectory "")
+			(outputdirectory "output/V2/")
 		)
 	)
@@
 			(unlocked yes)
 			(layer "F.SilkS")
+			(hide yes)
 			(effects
 				(font
@@
 			)
 		)
+		(sheetname "Root")
+		(sheetfile "radio433.kicad_sch")
 		(net_tie_pad_groups "1,2")
 		(fp_text user "IN"
@@
 		(layer "Edge.Cuts")
 	)
+	(gr_line
+		(start 253 105.5)
+		(end 257.49 101)
+		(stroke
+			(width 0.1)
+			(type default)
+		)
+		(layer "Edge.Cuts")
+	)
 	(gr_arc
 		(start 224.25 96)
@@
 	)
 	(gr_line
-		(start 257.49 105.5)
+		(start 253 105.5)
 		(end 224.25 105.5)
 		(stroke
@@
 	(gr_line
 		(start 257.49 80.19)
-		(end 257.49 105.5)
+		(end 257.49 101)
 		(stroke
 			(width 0.1)
@@
 	)
 	(via
-		(at 254.48 104.4)
-		(size 0.6)
-		(drill 0.3)
-		(layers "F.Cu" "B.Cu")
-		(free yes)
-		(net 1)
-	)
-	(via
 		(at 194.25 92.75)
 		(size 0.6)
@@
 	)
 	(via
-		(at 253.73 104.4)
-		(size 0.6)
-		(drill 0.3)
-		(layers "F.Cu" "B.Cu")
-		(free yes)
-		(net 1)
-	)
-	(via
 		(at 225.1 94.6)
 		(size 0.6)
@@
 		(size 0.6)
 		(drill 0.3)
-		(layers "F.Cu" "B.Cu")
-		(free yes)
-		(net 1)
-	)
-	(via
-		(at 254.48 103.65)
-		(size 0.6)
-		(drill 0.3)

Commit message: remover receiver
Parts:
- removed AE2: Antenna, radio433Lib:antenna_433_50R_helical
- removed C10, C11: 1p2, Capacitor_SMD:C_0603_1608Metric
- removed C12, C14: 100n, Capacitor_SMD:C_0603_1608Metric
- removed C13: 1u, Capacitor_SMD:C_0603_1608Metric
- removed C7, C8: 10p, Capacitor_SMD:C_0603_1608Metric
- removed C9: 4u7, Capacitor_SMD:C_0805_2012Metric
- removed J2: RX, Connector_PinHeader_2.54mm:PinHeader_1x07_P2.54mm_Vertical
- removed L3: 33n, Inductor_SMD:L_0603_1608Metric
- removed L4: 39n, Inductor_SMD:L_0603_1608Metric
- removed R3: 50k, Inductor_SMD:L_0603_1608Metric
- removed U2: MICRF219AAYQS, Package_SO:QSOP-16_3.9x4.9mm_P0.635mm
- removed Y2: 13M52313, Crystal:Crystal_SMD_3225-4Pin_3.2x2.5mm
- C6: value 100p -> 100p(100n)
- R1: value 100k -> 100k(22k)
Routing:
- net /VDD_RX: track 26.9 -> 0.00 mm, vias 2 -> 0
- net Net-(U2-RO1): track 14.0 -> 0.00 mm
- net GND: track 15.0 -> 2.04 mm, vias 40 -> 27
- net /SCLK: track 12.2 -> 0.00 mm, vias 2 -> 0
- net /RSSI: track 11.7 -> 0.00 mm, vias 2 -> 0
- net /DOUT: track 11.1 -> 0.00 mm
- net /SHDN: track 10.8 -> 0.00 mm
- net Net-(U2-CAGC): track 9.97 -> 0.00 mm, vias 2 -> 0
- net /ANT_CC: track 8.19 -> 0.00 mm
- net Net-(U2-RO2): track 6.78 -> 0.00 mm
- net /ANT: track 5.71 -> 0.00 mm
- net Net-(U2-CTH): track 5.36 -> 0.00 mm
- net /ANT_C: track 1.93 -> 0.00 mm
Other:
- board text removed: "CLK"
- board text removed: "DOUT"
- board text removed: "RSSI"
- board text removed: "SHDN"

Commit message: V3
Parts:
- added AE3: Antenna_Shield, Connector_PinSocket_2.54mm:PinSocket_1x02_P2.54mm_Vertical, F.Cu at (199.8, 95.5)
- added C10: 2p7, Capacitor_SMD:C_0603_1608Metric, F.Cu at (206.4, 95.4)
- added C11: 6p2, Capacitor_SMD:C_0603_1608Metric, F.Cu at (204.0, 96.2)
- added C7: 1n, Capacitor_SMD:C_0603_1608Metric, F.Cu at (210.4, 100.2)
- added C8: 100nF, Capacitor_SMD:C_0805_2012Metric, F.Cu at (208.4, 100.0)
- added C9: NC, Capacitor_SMD:C_0603_1608Metric, F.Cu at (208.8, 96.2)
- added J2: RX, Connector_PinHeader_2.54mm:PinHeader_1x05_P2.54mm_Vertical, F.Cu at (210.8, 103.5)
- added L3: 33nH, Inductor_SMD:L_0603_1608Metric, F.Cu at (210.4, 96.2)
- added L4: 22nH, Inductor_SMD:L_0603_1608Metric, F.Cu at (202.4, 96.2)
- added R3: 10k, Resistor_SMD:R_0603_1608Metric, F.Cu at (218.7, 100.6)
- added U2: CMT2210LC, Package_SO:SO-8_3.9x4.9mm_P1.27mm, F.Cu at (214.3, 98.0)
- added Y2: 27M1383, Crystal:Crystal_SMD_3225-4Pin_3.2x2.5mm, F.Cu at (219.4, 95.8)
- Logo1, Logo2: moved to B.Cu
- moved Logo2 11.6 mm to (210.8, 97.0), turned to 180 degrees
- moved Logo1 9.75 mm to (239.4, 96.8), turned to 180 degrees
Connections:
- net /VDD_TX renamed /VDD
Routing:
- net /VDD: track 32.8 -> 65.4 mm
- net /SHDN: track 0.00 -> 13.6 mm, vias 0 -> 1
- net Net-(AE3-A): track 0.00 -> 5.90 mm
- net /DOUT: track 0.00 -> 5.88 mm
- net Net-(U2-XIN): track 0.00 -> 5.78 mm
- net Net-(U2-RFIN): track 0.00 -> 5.18 mm
- net GND: vias 27 -> 58
Other:
- board size 70.5 x 26.8 mm -> 59.9 x 26.8 mm
